Commit message: add launch file for checking urdf

File: ken_description/urdf/ken.xacro (robot description, xacro)
@@ -8,40 +8,28 @@
   </material>
   <link name="base_link"/>
-  <link name="${NAME_LINK_BASE}">
+  <link name="arm_base_link">
     <visual>
       <origin xyz="0 0 0" rpy="0 0 0"/>
       <geometry>
-        <mesh filename="package://${MESH_LINK_BASE}"
-            scale="1 1 1"/>
+        <mesh filename="package://ken_description/meshes/arm_base.stl" scale="1 1 1"/>
       </geometry>
-      <material name="black"/>
+      <material name="grey"/>
     </visual>
     <collision>
       <origin xyz="0 0 0" rpy="0 0 0"/>
       <geometry>
-        <mesh filename="package://${MESH_COLLISION_LINK_BASE}"
-            scale="1 1 1"/>
+        <mesh filename="package://ken_description/meshes/arm_base.stl" scale="1 1 1"/>
       </geometry>
-      <material name="black"/>
     </collision>
     <inertial>
-      <mass value="0.06645"/>
-      <origin xyz="-1.31E-02 7.00E-06 2.12E-02" rpy="0 ${M_PI/8} 0"/>
-      <inertia ixx="1.66E-05" ixy="1.80E-09" ixz="-5.75E-07" iyy="2.36E-05" iyz="-3.23E-08" izz="1.77E-05"/>
+      <mass value="0.3"/>
+      <origin xyz="0.0 0.0 0.0" rpy="0 0 0"/>
+      <inertia ixx="0.1" ixy="0.1" ixz="0.1" iyy="0.1" iyz="0.1" izz="0.1"/>
     </inertial>
   </link>
-  <joint name="${NAME_JOINT_1}" type="revolute">
+  <joint name="base_to_arm_base" type="fixed">
     <origin xyz="0 0 0.0454" rpy="0 0 0"/>
-    <axis xyz="0 0 1"/>
-    <limit
-      effort="10.0"
-      velocity="${joints_vlimit}"
-      lower="${joint1_lower_limit}"
-      upper="${joint1_upper_limit}"
-      />
-    <parent link="${NAME_LINK_BASE}"/>
-    <child link="${NAME_LINK_1}"/>
-    <dynamics damping="1.0e-6" friction="2.0e-1"/>
+    <parent link="base_link"/>
+    <child link="arm_base_link"/>
   </joint>
-  </xacro:macro>
 </robot>

Commit message: update stl

File: ken_description/urdf/ken.xacro (robot description, xacro)
@@ -8,4 +8,9 @@
   </material>
   <link name="base_link"/>
+  <joint name="base_to_arm_base" type="fixed">
+    <origin xyz="0 0 0.0" rpy="0 0 0"/>
+    <parent link="base_link"/>
+    <child link="arm_base_link"/>
+  </joint>
   <link name="arm_base_link">
     <visual>
@@ -28,8 +33,3 @@
     </inertial>
   </link>
-  <joint name="base_to_arm_base" type="fixed">
-    <origin xyz="0 0 0.0454" rpy="0 0 0"/>
-    <parent link="base_link"/>
-    <child link="arm_base_link"/>
-  </joint>
 </robot>

Commit message: add other links

File: ken_description/urdf/ken.xacro (robot description, xacro)
@@ -24,4 +24,32 @@
     <parent link="arm_base_link"/>
     <child link="arm_link1"/>
+    <limit effort="${joint_effort_limit}" velocity="${joint_velocity_limit}" lower="${-90*TO_RADIAN}" upper="${90*TO_RADIAN}" />
+  </joint>
+  <joint name="arm_link1_to_arm_link2" type="revolute">
+    <origin xyz="0.015 -0.019 0.023" rpy="0 0 0"/>
+    <axis xyz="0 1 0"/>
+    <parent link="arm_link1"/>
+    <child link="arm_link2"/>
+    <limit effort="${joint_effort_limit}" velocity="${joint_velocity_limit}" lower="${-90*TO_RADIAN}" upper="${90*TO_RADIAN}" />
+  </joint>
+  <joint name="arm_link2_to_arm_link3" type="revolute">
+    <origin xyz="0.1 0.0 0.0" rpy="0 0 0"/>
+    <axis xyz="0 1 0"/>
+    <parent link="arm_link2"/>
+    <child link="arm_link3"/>
+    <limit effort="${joint_effort_limit}" velocity="${joint_velocity_limit}" lower="${-90*TO_RADIAN}" upper="${90*TO_RADIAN}" />
+  </joint>
+  <joint name="arm_link3_to_arm_link4" type="revolute">
+    <origin xyz="0.125 0.0 0.0" rpy="0 0 0"/>
+    <axis xyz="0 1 0"/>
+    <parent link="arm_link3"/>
+    <child link="arm_link4"/>
+    <limit effort="${joint_effort_limit}" velocity="${joint_velocity_limit}" lower="${-90*TO_RADIAN}" upper="${90*TO_RADIAN}" />
+  </joint>
+  <joint name="arm_link4_to_shinai_link" type="revolute">
+    <origin xyz="0.067 0.014 -0.02" rpy="0 0 0"/>
+    <axis xyz="1 0 0"/>
+    <parent link="arm_link4"/>
+    <child link="shinai_link"/>
     <limit effort="${joint_effort_limit}" velocity="${joint_velocity_limit}" lower="${-90*TO_RADIAN}" upper="${90*TO_RADIAN}" />
   </joint>
@@ -66,3 +94,83 @@
     </inertial>
   </link>
+  <link name="arm_link2">
+    <visual>
+      <origin xyz="0 0 0" rpy="0 0 0"/>
+      <geometry>
+        <mesh filename="package://ken_description/meshes/link2.stl" scale="1 1 1"/>
+      </geometry>
+      <material name="grey"/>
+    </visual>
+    <collision>
+      <origin xyz="0 0 0" rpy="0 0 0"/>
+      <geometry>
+        <mesh filename="package://ken_description/meshes/link2.stl" scale="1 1 1"/>
+      </geometry>
+    </collision>
+    <inertial>
+      <mass value="0.3"/>
+      <origin xyz="0.0 0.0 0.0" rpy="0 0 0"/>
+      <inertia ixx="0.1" ixy="0.1" ixz="0.1" iyy="0.1" iyz="0.1" izz="0.1"/>
+    </inertial>
+  </link>
+  <link name="arm_link3">
+    <visual>
+      <origin xyz="0 0 0" rpy="0 -${pi/2} 0"/>
+      <geometry>
+        <mesh filename="package://ken_description/meshes/link3.stl" scale="1 1 1"/>
+      </geometry>
+      <material name="white"/>
+    </visual>
+    <collision>
+      <origin xyz="0 0 0" rpy="0 -${pi/2} 0"/>
+      <geometry>
+        <mesh filename="package://ken_description/meshes/link3.stl" scale="1 1 1"/>
+      </geometry>
+    </collision>
+    <inertial>
+      <mass value="0.3"/>
+      <origin xyz="0.0 0.0 0.0" rpy="0 0 0"/>
+      <inertia ixx="0.1" ixy="0.1" ixz="0.1" iyy="0.1" iyz="0.1" izz="0.1"/>
+    </inertial>
+  </link>
+  <link name="arm_link4">
+    <visual>
+      <origin xyz="0 0 0" rpy="0 -${pi/2} 0"/>
+      <geometry>
+        <mesh filename="package://ken_description/meshes/link4.stl" scale="1 1 1"/>
+      </geometry>
+      <material name="grey"/>
+    </visual>
+    <collision>
+      <origin xyz="0 0 0" rpy="0 -${pi/2} 0"/>
+      <geometry>
+        <mesh filename="package://ken_description/meshes/link4.stl" scale="1 1 1"/>
+      </geometry>
+    </collision>
+    <inertial>
+      <mass value="0.3"/>
+      <origin xyz="0.0 0.0 0.0" rpy="0 0 0"/>
+      <inertia ixx="0.1" ixy="0.1" ixz="0.1" iyy="0.1" iyz="0.1" izz="0.1"/>
+    </inertial>
+  </link>
+  <link name="shinai_link">
+    <visual>
+      <origin xyz="0 0 0" rpy="0 0 0"/>
+      <geometry>
+        <mesh filename="package://ken_description/meshes/shinai.stl" scale="1 1 1"/>
+      </geometry>
+      <material name="white"/>
+    </visual>
+    <collision>
+      <origin xyz="0 0 0" rpy="0 0 0"/>
+      <geometry>
+        <mesh filename="package://ken_description/meshes/shinai.stl" scale="1 1 1"/>
+      </geometry>
+    </collision>
+    <inertial>
+      <mass value="0.3"/>
+      <origin xyz="0.0 0.0 0.0" rpy="0 0 0"/>
+      <inertia ixx="0.1" ixy="0.1" ixz="0.1" iyy="0.1" iyz="0.1" izz="0.1"/>
+    </inertial>
+  </link>
 </robot>

Commit message: change joint limit angle

File: ken_description/urdf/ken.xacro (robot description, xacro)
@@ -24,5 +24,5 @@
     <parent link="arm_base_link"/>
     <child link="arm_link1"/>
-    <limit effort="${joint_effort_limit}" velocity="${joint_velocity_limit}" lower="${-90*TO_RADIAN}" upper="${90*TO_RADIAN}" />
+    <limit effort="${joint_effort_limit}" velocity="${joint_velocity_limit}" lower="${-180*TO_RADIAN}" upper="${180*TO_RADIAN}" />
   </joint>
   <joint name="arm_link1_to_arm_link2" type="revolute">
@@ -31,5 +31,5 @@
     <parent link="arm_link1"/>
     <child link="arm_link2"/>
-    <limit effort="${joint_effort_limit}" velocity="${joint_velocity_limit}" lower="${-90*TO_RADIAN}" upper="${90*TO_RADIAN}" />
+    <limit effort="${joint_effort_limit}" velocity="${joint_velocity_limit}" lower="${-180*TO_RADIAN}" upper="${10*TO_RADIAN}" />
   </joint>
   <joint name="arm_link2_to_arm_link3" type="revolute">
@@ -38,5 +38,5 @@
     <parent link="arm_link2"/>
     <child link="arm_link3"/>
-    <limit effort="${joint_effort_limit}" velocity="${joint_velocity_limit}" lower="${-90*TO_RADIAN}" upper="${90*TO_RADIAN}" />
+    <limit effort="${joint_effort_limit}" velocity="${joint_velocity_limit}" lower="${-150*TO_RADIAN}" upper="${150*TO_RADIAN}" />
   </joint>
   <joint name="arm_link3_to_arm_link4" type="revolute">
@@ -52,5 +52,5 @@
     <parent link="arm_link4"/>
     <child link="shinai_link"/>
-    <limit effort="${joint_effort_limit}" velocity="${joint_velocity_limit}" lower="${-90*TO_RADIAN}" upper="${90*TO_RADIAN}" />
+    <limit effort="${joint_effort_limit}" velocity="${joint_velocity_limit}" lower="${-180*TO_RADIAN}" upper="${180*TO_RADIAN}" />
   </joint>
   <link name="arm_base_link">

Commit message: change for dh param

File: ken_description/urdf/ken.xacro (robot description, xacro)
@@ -15,10 +15,10 @@
   <link name="base_link"/>
   <joint name="base_to_arm_base" type="fixed">
-    <origin xyz="0 0 0.0" rpy="0 0 0"/>
+    <origin xyz="0 0 0.065" rpy="0 0 0"/>
     <parent link="base_link"/>
     <child link="arm_base_link"/>
   </joint>
   <joint name="arm_base_to_arm_link1" type="revolute">
-    <origin xyz="0 0 0.042" rpy="0 0 0"/>
+    <origin xyz="0 0 0" rpy="0 0 0"/>
     <axis xyz="0 0 1"/>
     <parent link="arm_base_link"/>
@@ -27,13 +27,13 @@
   </joint>
   <joint name="arm_link1_to_arm_link2" type="revolute">
-    <origin xyz="0.015 -0.019 0.023" rpy="0 0 0"/>
-    <axis xyz="0 1 0"/>
+    <origin xyz="0.015 -0.02 0.0" rpy="${pi/2} 0 0"/>
+    <axis xyz="0 0 1"/>
     <parent link="arm_link1"/>
     <child link="arm_link2"/>
-    <limit effort="${joint_effort_limit}" velocity="${joint_velocity_limit}" lower="${-180*TO_RADIAN}" upper="${10*TO_RADIAN}" />
+    <limit effort="${joint_effort_limit}" velocity="${joint_velocity_limit}" lower="${-10*TO_RADIAN}" upper="${180*TO_RADIAN}" />
   </joint>
   <joint name="arm_link2_to_arm_link3" type="revolute">
     <origin xyz="0.1 0.0 0.0" rpy="0 0 0"/>
-    <axis xyz="0 1 0"/>
+    <axis xyz="0 0 1"/>
     <parent link="arm_link2"/>
     <child link="arm_link3"/>
@@ -41,6 +41,6 @@
   </joint>
   <joint name="arm_link3_to_arm_link4" type="revolute">
-    <origin xyz="0.125 0.0 0.0" rpy="0 0 0"/>
-    <axis xyz="0 1 0"/>
+    <origin xyz="0.125 0.0 -0.014" rpy="0 0 ${-pi/2}"/>
+    <axis xyz="0 0 1"/>
     <parent link="arm_link3"/>
     <child link="arm_link4"/>
@@ -48,6 +48,6 @@
   </joint>
   <joint name="arm_link4_to_shinai_link" type="revolute">
-    <origin xyz="0.067 0.014 -0.02" rpy="0 0 0"/>
-    <axis xyz="1 0 0"/>
+    <origin xyz="0.016 0.075 0.0" rpy="${pi/2} 0 ${pi}"/>
+    <axis xyz="0 0 1"/>
     <parent link="arm_link4"/>
     <child link="shinai_link"/>
@@ -56,5 +56,5 @@
   <link name="arm_base_link">
     <visual>
-      <origin xyz="0 0 0" rpy="0 0 0"/>
+      <origin xyz="0 0 -0.065" rpy="0 0 0"/>
       <geometry>
         <mesh filename="package://ken_description/meshes/arm_base.stl" scale="1 1 1"/>
@@ -63,5 +63,5 @@
     </visual>
     <collision>
-      <origin xyz="0 0 0" rpy="0 0 0"/>
+      <origin xyz="0 0 -0.065" rpy="0 0 0"/>
       <geometry>
         <mesh filename="package://ken_description/meshes/arm_base.stl" scale="1 1 1"/>
@@ -76,5 +76,5 @@
   <link name="arm_link1">
     <visual>
-      <origin xyz="0 0 0" rpy="0 0 0"/>
+      <origin xyz="0 0 -0.023" rpy="0 0 0"/>
       <geometry>
         <mesh filename="package://ken_description/meshes/link1.stl" scale="1 1 1"/>
@@ -83,5 +83,5 @@
     </visual>
     <collision>
-      <origin xyz="0 0 0" rpy="0 0 0"/>
+      <origin xyz="0 0 -0.023" rpy="0 0 0"/>
       <geometry>
         <mesh filename="package://ken_description/meshes/link1.stl" scale="1 1 1"/>
@@ -96,5 +96,5 @@
   <link name="arm_link2">
     <visual>
-      <origin xyz="0 0 0" rpy="0 0 0"/>
+      <origin xyz="0 0 0" rpy="${-pi/2} 0 0"/>
       <geometry>
         <mesh filename="package://ken_description/meshes/link2.stl" scale="1 1 1"/>
@@ -103,5 +103,5 @@
     </visual>
     <collision>
-      <origin xyz="0 0 0" rpy="0 0 0"/>
+      <origin xyz="0 0 0" rpy="${-pi/2} 0 0"/>
       <geometry>
         <mesh filename="package://ken_description/meshes/link2.stl" scale="1 1 1"/>
@@ -116,5 +116,5 @@
   <link name="arm_link3">
     <visual>
-      <origin xyz="0 0 0" rpy="0 -${pi/2} 0"/>
+      <origin xyz="0 0 0" rpy="${-pi/2} 0 ${pi/2}"/>
       <geometry>
         <mesh filename="package://ken_description/meshes/link3.stl" scale="1 1 1"/>
@@ -123,5 +123,5 @@
     </visual>
     <collision>
-      <origin xyz="0 0 0" rpy="0 -${pi/2} 0"/>
+      <origin xyz="0 0 0" rpy="${-pi/2} 0 ${pi/2}"/>
       <geometry>
         <mesh filename="package://ken_description/meshes/link3.stl" scale="1 1 1"/>
@@ -136,5 +136,5 @@
   <link name="arm_link4">
     <visual>
-      <origin xyz="0 0 0" rpy="0 -${pi/2} 0"/>
+      <origin xyz="0 0 0.014" rpy="${-pi/2} 0 ${pi}"/>
       <geometry>
         <mesh filename="package://ken_description/meshes/link4.stl" scale="1 1 1"/>
@@ -143,5 +143,5 @@
     </visual>
     <collision>
-      <origin xyz="0 0 0" rpy="0 -${pi/2} 0"/>
+      <origin xyz="0 0 0.014" rpy="${-pi/2} 0 ${pi}"/>
       <geometry>
         <mesh filename="package://ken_description/meshes/link4.stl" scale="1 1 1"/>
@@ -156,5 +156,5 @@
   <link name="shinai_link">
     <visual>
-      <origin xyz="0 0 0" rpy="0 0 0"/>
+      <origin xyz="0 0 0" rpy="${pi/2} 0 ${pi/2}"/>
       <geometry>
         <mesh filename="package://ken_description/meshes/shinai.stl" scale="1 1 1"/>
@@ -163,5 +163,5 @@
     </visual>
     <collision>
-      <origin xyz="0 0 0" rpy="0 0 0"/>
+      <origin xyz="0 0 0" rpy="${pi/2} 0 ${pi/2}"/>
       <geometry>
         <mesh filename="package://ken_description/meshes/shinai.stl" scale="1 1 1"/>

Commit message: add tip link

File: ken_description/urdf/ken.xacro (robot description, xacro)
@@ -14,4 +14,5 @@
   <xacro:property name="TO_RADIAN" value="${pi / 180.0}"/>
   <link name="base_link"/>
+  <link name="tip_link"/>
   <joint name="base_to_arm_base" type="fixed">
     <origin xyz="0 0 0.065" rpy="0 0 0"/>
@@ -53,4 +54,9 @@
     <child link="shinai_link"/>
     <limit effort="${joint_effort_limit}" velocity="${joint_velocity_limit}" lower="${-180*TO_RADIAN}" upper="${180*TO_RADIAN}" />
+  </joint>
+  <joint name="shinai_link_to_tip" type="fixed">
+    <origin xyz="0.31 0 0" rpy="0 0 0"/>
+    <parent link="shinai_link"/>
+    <child link="tip_link"/>
   </joint>
   <link name="arm_base_link">
