Commit message: add first link

File: ken_description/urdf/ken.urdf.xacro (robot description, xacro)
@@ -7,5 +7,3 @@
     <child link="base_link"/>
   </joint>
-  <xacro:property name="M_PI" value="3.14159"/>
-  <xacro:property name="TO_RADIAN" value="${M_PI / 180.0}"/>
 </robot>

File: ken_description/urdf/ken.xacro (robot description, xacro)
@@ -5,6 +5,12 @@
   </material>
   <material name="grey">
-    <color rgba="0.3 0.3 0.3 1.0"/>
+    <color rgba="0.4 0.4 0.4 1.0"/>
   </material>
+  <material name="white">
+    <color rgba="0.9 0.9 0.9 1.0"/>
+  </material>
+  <xacro:property name="joint_effort_limit" value="10.0"/>
+  <xacro:property name="joint_velocity_limit" value="1.0"/>
+  <xacro:property name="TO_RADIAN" value="${pi / 180.0}"/>
   <link name="base_link"/>
   <joint name="base_to_arm_base" type="fixed">
@@ -12,4 +18,11 @@
     <parent link="base_link"/>
     <child link="arm_base_link"/>
+  </joint>
+  <joint name="arm_base_to_arm_link1" type="revolute">
+    <origin xyz="0 0 0.042" rpy="0 0 0"/>
+    <axis xyz="0 0 1"/>
+    <parent link="arm_base_link"/>
+    <child link="arm_link1"/>
+    <limit effort="${joint_effort_limit}" velocity="${joint_velocity_limit}" lower="${-90*TO_RADIAN}" upper="${90*TO_RADIAN}" />
   </joint>
   <link name="arm_base_link">
@@ -33,3 +46,23 @@
     </inertial>
   </link>
+  <link name="arm_link1">
+    <visual>
+      <origin xyz="0 0 0" rpy="0 0 0"/>
+      <geometry>
+        <mesh filename="package://ken_description/meshes/link1.stl" scale="1 1 1"/>
+      </geometry>
+      <material name="white"/>
+    </visual>
+    <collision>
+      <origin xyz="0 0 0" rpy="0 0 0"/>
+      <geometry>
+        <mesh filename="package://ken_description/meshes/link1.stl" scale="1 1 1"/>
+      </geometry>
+    </collision>
+    <inertial>
+      <mass value="0.3"/>
+      <origin xyz="0.0 0.0 0.0" rpy="0 0 0"/>
+      <inertia ixx="0.1" ixy="0.1" ixz="0.1" iyy="0.1" iyz="0.1" izz="0.1"/>
+    </inertial>
+  </link>
 </robot>

Commit message: add d435 frame to robot xacro

File: ken_description/urdf/ken.urdf.xacro (robot description, xacro)
@@ -7,3 +7,33 @@
     <child link="base_link"/>
   </joint>
+  <!-- The following values model the aluminum peripherial case for the
+  D435 camera, with the camera joint represented by the actual
+  peripherial camera tripod mount -->
+  <xacro:property name="d435_cam_width" value="0.090"/>
+  <xacro:property name="d435_cam_height" value="0.025"/>
+  <xacro:property name="d435_cam_depth" value="0.02505"/>
+  <xacro:property name="d435_cam_mount_from_center_offset" value="0.0149"/>
+  <!-- glass cover is 0.1 mm inwards from front aluminium plate -->
+  <xacro:property name="d435_glass_to_front" value="0.1e-3"/>
+  <!-- see datasheet Revision 007, Fig. 4-4 page 65 -->
+  <xacro:property name="d435_zero_depth_to_glass" value="4.2e-3"/>
+  <!-- convenience precomputation to avoid clutter-->
+  <xacro:property name="d435_mesh_x_offset" value="${d435_cam_mount_from_center_offset-d435_glass_to_front-d435_zero_depth_to_glass}"/>
+  <!-- The following offset is relative the the physical D435 camera peripherial
+  camera tripod mount -->
+  <xacro:property name="d435_cam_depth_px" value="${d435_cam_mount_from_center_offset}"/>
+  <xacro:property name="d435_cam_depth_py" value="0.0175"/>
+  <xacro:property name="d435_cam_depth_pz" value="${d435_cam_height/2}"/>
+  <link name="camera_link"/>
+  <link name="camera_bottom_screw_frame"/>
+  <joint name="camera_link_joint" type="fixed">
+    <origin xyz="${d435_mesh_x_offset} ${d435_cam_depth_py} ${d435_cam_depth_pz}" rpy="0 0 0"/>
+    <parent link="camera_bottom_screw_frame"/>
+    <child link="camera_link" />
+  </joint>
+  <joint name="base_link_to_camera_bottom_screw_frame" type="fixed">
+    <origin xyz="-0.134856 -0.07 0.381814" rpy="0 ${pi*18/180} 0"/>
+    <parent link="base_link"/>
+    <child link="camera_bottom_screw_frame"/>
+  </joint>
 </robot>

Commit message: change pos

File: ken_description/urdf/ken.urdf.xacro (robot description, xacro)
@@ -33,5 +33,5 @@
   </joint>
   <joint name="base_link_to_camera_bottom_screw_frame" type="fixed">
-    <origin xyz="-0.134856 -0.07 0.381814" rpy="0 ${pi*18/180} 0"/>
+    <origin xyz="-0.114856 -0.07 0.381814" rpy="0 ${pi*18/180} 0"/>
     <parent link="base_link"/>
     <child link="camera_bottom_screw_frame"/>
